File: A ducking ruler/A ducking ruler.kicad_pcb (KiCad board)
At the start: 2 copper layers, 210 x 40 mm, 32 parts

Commit message: feat: added ducks
Parts:
- added G***: LOGO, Angelussss:Doodle_Duck, F.Cu at (233.0, 97.0)
- added G***: LOGO, Angelussss:Basic_Duck, F.Cu at (131.0, 98.0)
- added G***: LOGO, Angelussss:Dino_Duck, F.Cu at (187.0, 106.0)
